File: laser_carousel/Sensor Carousel.sch (EAGLE design)
At the start: 50 parts

Commit message: More Board Committs
Parts:
- added JP1: (no value), adafruit:PINHD-1X6
- added JP2: (no value), adafruit:PINHD-1X3
- added MGT1, MGT2: MOUNTING_HOLE, ENGI301:MOUNTING_HOLE
- C1, C12, C2, C4, C8: device adafruit:C-US050-024X044 -> adafruit:C-US025-024X044
- C10, C11, C13, C14, C15, C16, C3, C5, C6, C7, C9: device adafruit:C-US050-025X075 -> adafruit:C-US025-024X044
- R1, R10, R11, R12, R13, R14, R15, R16, R2, R3, R4, R5, R6, R7, R8, R9: device adafruit:R-US_0204/7 -> adafruit:R-US_0204/2V
Connections:
- removed net N$1: C1.1, U$1.GND
- removed net N$10: C4.1, U$4.GND
- removed net N$11: C4.2, R4.1, U$4.VCC
- removed net N$12: R4.2, U$4.OUT
- removed net N$13: C5.1, U$5.GND
- removed net N$14: C5.2, R5.1, U$5.VCC
- removed net N$15: R5.2, U$5.OUT
- removed net N$16: C6.1, U$6.GND
- removed net N$17: C6.2, R6.1, U$6.VCC
- removed net N$18: R6.2, U$6.OUT
- removed net N$19: C7.1, U$7.GND
- removed net N$2: C1.2, R1.1, U$1.VCC
- removed net N$20: C7.2, R7.1, U$7.VCC
- removed net N$21: R7.2, U$7.OUT
- removed net N$22: C8.1, U$8.GND
- removed net N$23: C8.2, R8.1, U$8.VCC
- removed net N$24: R8.2, U$8.OUT
- removed net N$25: C9.1, U$9.GND
- removed net N$26: C9.2, R9.1, U$9.VCC
- removed net N$27: R9.2, U$9.OUT
- removed net N$28: C10.1, U$10.GND
- removed net N$29: C10.2, R10.1, U$10.VCC
- removed net N$3: R1.2, U$1.OUT
- removed net N$30: R10.2, U$10.OUT
- removed net N$31: C11.1, U$11.GND
- removed net N$32: C11.2, R11.1, U$11.VCC
- removed net N$33: R11.2, U$11.OUT
- removed net N$34: C12.1, U$12.GND
- removed net N$35: C12.2, R12.1, U$12.VCC
- removed net N$36: R12.2, U$12.OUT
- removed net N$37: C13.1, U$13.GND
- removed net N$38: C13.2, R13.1, U$13.VCC
- removed net N$39: R13.2, U$13.OUT
- removed net N$4: C2.1, U$2.GND
- removed net N$40: C14.1, U$14.GND
- removed net N$41: C14.2, R14.1, U$14.VCC
- removed net N$42: R14.2, U$14.OUT
- removed net N$43: C15.1, U$15.GND
- removed net N$44: C15.2, R15.1, U$15.VCC
- removed net N$45: R15.2, U$15.OUT
- removed net N$46: C16.1, U$16.GND
- removed net N$47: C16.2, R16.1, U$16.VCC
- removed net N$48: R16.2, U$16.OUT
- removed net N$5: C2.2, R2.1, U$2.VCC
- removed net N$6: R2.2, U$2.OUT
- removed net N$7: C3.1, U$3.GND
- removed net N$8: C3.2, R3.1, U$3.VCC
- removed net N$9: R3.2, U$3.OUT
- new net A0: IC1.S0, IC2.S2, JP2.1
- new net A1: IC1.S1, IC2.S1, JP2.2
- new net A2: IC1.S2, IC2.S0, JP2.3
- new net GND: C1.1, C10.1, C11.1, C12.1, C13.1, C14.1, C15.1, C16.1, C2.1, C3.1, C4.1, C5.1, C6.1, C7.1, C8.1, C9.1, IC1.E, IC1.GND, IC2.E, IC2.GND, JP1.5, JP1.6, U$1.GND, U$10.GND, U$11.GND, U$12.GND, U$13.GND, U$14.GND, U$15.GND, U$16.GND, U$2.GND, U$3.GND, U$4.GND, U$5.GND, U$6.GND, U$7.GND, U$8.GND, U$9.GND
- new net U1: IC2.I0, R1.2, U$1.OUT
- new net U10: IC2.I7, R10.2, U$10.OUT
- new net U11: IC2.I3, R11.2, U$11.OUT
- new net U12: IC2.I5, R12.2, U$12.OUT
- new net U13: IC2.I1, R13.2, U$13.OUT
- new net U14: IC2.I6, R14.2, U$14.OUT
- new net U15: IC2.I2, R15.2, U$15.OUT
- new net U16: IC2.I4, R16.2, U$16.OUT
- new net U2: IC1.I7, R2.2, U$2.OUT
- new net U3: IC1.I6, R3.2, U$3.OUT
- new net U4: IC1.I5, R4.2, U$4.OUT
- new net U5: IC1.I4, R5.2, U$5.OUT
- new net U6: IC1.I3, R6.2, U$6.OUT
- new net U7: IC1.I2, R7.2, U$7.OUT
- new net U8: IC1.I1, R8.2, U$8.OUT
- new net U9: IC1.I0, R9.2, U$9.OUT
- new net VIN_5V: C1.2, C10.2, C11.2, C12.2, C13.2, C14.2, C15.2, C16.2, C2.2, C3.2, C4.2, C5.2, C6.2, C7.2, C8.2, C9.2, IC1.VCC, IC2.VCC, JP1.1, JP1.2, R1.1, R10.1, R11.1, R12.1, R13.1, R14.1, R15.1, R16.1, R2.1, R3.1, R4.1, R5.1, R6.1, R7.1, R8.1, R9.1, U$1.VCC, U$10.VCC, U$11.VCC, U$12.VCC, U$13.VCC, U$14.VCC, U$15.VCC, U$16.VCC, U$2.VCC, U$3.VCC, U$4.VCC, U$5.VCC, U$6.VCC, U$7.VCC, U$8.VCC, U$9.VCC
- new net Y1: IC1.Y, JP1.3
- new net Y2: IC2.Y, JP1.4
