File: laser_carousel/carousel.brd (EAGLE design)
At the start: 63.5 x 63.5 mm, 50 parts

Commit message: Carousel PCB Updates
Parts:
- added JP1: (no value), adafruit:1X06
- added JP2: (no value), adafruit:1X03
- moved IC2 19.1 mm to (6.60, -6.35), turned to 90 degrees
- moved IC1 19.0 mm to (-6.60, 6.35), turned to 270 degrees
Connections:
- removed net N$12: R4.2, U$4.P$2
- removed net N$15: R5.2, U$5.P$2
- removed net N$18: R6.2, U$6.P$2
- removed net N$2: R13.2, U$13.P$2
- removed net N$21: R7.2, U$7.P$2
- removed net N$24: R8.2, U$8.P$2
- removed net N$27: R9.2, U$9.P$2
- removed net N$3: R1.2, U$1.P$2
- removed net N$30: R10.2, U$10.P$2
- removed net N$33: R11.2, U$11.P$2
- removed net N$36: R12.2, U$12.P$2
- removed net N$42: R14.2, U$14.P$2
- removed net N$45: R15.2, U$15.P$2
- removed net N$48: R16.2, U$16.P$2
- removed net N$6: R2.2, U$2.P$2
- removed net N$9: R3.2, U$3.P$2
- new net A0: IC1.11, IC2.9, JP2.1
- new net A1: IC1.10, IC2.10, JP2.2
- new net A2: IC1.9, IC2.11, JP2.3
- new net U1: IC2.4, R1.2, U$1.P$2
- new net U10: IC2.12, R10.2, U$10.P$2
- new net U11: IC2.1, R11.2, U$11.P$2
- new net U12: IC2.14, R12.2, U$12.P$2
- new net U13: IC2.3, R13.2, U$13.P$2
- new net U14: IC2.13, R14.2, U$14.P$2
- new net U15: IC2.2, R15.2, U$15.P$2
- new net U16: IC2.15, R16.2, U$16.P$2
- new net U2: IC1.12, R2.2, U$2.P$2
- new net U3: IC1.13, R3.2, U$3.P$2
- new net U4: IC1.14, R4.2, U$4.P$2
- new net U5: IC1.15, R5.2, U$5.P$2
- new net U6: IC1.1, R6.2, U$6.P$2
- new net U7: IC1.2, R7.2, U$7.P$2
- new net U8: IC1.3, R8.2, U$8.P$2
- new net U9: IC1.4, R9.2, U$9.P$2
- new net Y1: IC1.5, JP1.3
- new net Y2: IC2.5, JP1.4
- net GND: now also JP1.5, JP1.6
- net VIN_5V: now also JP1.1, JP1.2
Routing:
- net U2: track 0.00 -> 64.5 mm
- net U11: track 0.00 -> 59.6 mm
- net U13: track 0.00 -> 46.4 mm
- net U16: track 0.00 -> 34.1 mm
- net U10: track 0.00 -> 30.4 mm
- net U3: track 0.00 -> 27.6 mm
- net VIN_5V: track 0.00 -> 24.8 mm
- net U4: track 0.00 -> 21.0 mm
- net U12: track 0.00 -> 21.0 mm
- net U14: track 0.00 -> 20.9 mm
- net Y1: track 0.00 -> 20.9 mm
- net U9: track 0.00 -> 20.2 mm
- net U1: track 0.00 -> 20.2 mm
- net Y2: track 0.00 -> 16.7 mm
- net U8: track 0.00 -> 16.0 mm
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
Commit message: More Board Committs
Parts:
- added FUD1, FUD2, FUD3, FUD4: FIDUCIAL, ENGI301:FIDUCIAL_40MIL
- added MGT1, MGT2: MOUNTING_HOLE, ENGI301:MOUNTING_HOLE
- C12: device adafruit:C050-024X044 -> adafruit:C025-024X044
- moved R9 1.27 mm to (-21.8, -1.27)
- moved R1 1.02 mm to (22.1, 1.27)
- moved R7 0.81 mm to (-16.9, 14.9)
- moved R8 0.74 mm to (-21.2, 7.45)
- moved R11 0.72 mm to (-14.9, -16.7)
Connections:
- removed net N$10: C4.1, U$4.P$3
- removed net N$4: C2.1, U$2.P$3
- removed net N$7: C3.1, U$3.P$3
- net GND: now also C2.1, C3.1, C4.1, U$2.P$3, U$3.P$3, U$4.P$3
Routing:
- net GND: track 2.14 -> 86.5 mm, vias 0 -> 1
- net VIN_5V: track 24.8 -> 94.3 mm, vias 0 -> 2
- net U2: track 64.5 -> 30.8 mm, vias 0 -> 2
- net U11: track 59.6 -> 32.7 mm, vias 0 -> 2
- net U13: track 46.4 -> 24.1 mm
- net U16: track 34.1 -> 24.8 mm
- net N$4: track 2.20 -> 0.00 mm
- net N$7: track 2.14 -> 0.00 mm
- net U14: vias 0 -> 1
- added copper zone on layer 16, net GND
- added copper zone on layer 16, net VIN_5V
Other:
- board text added: "407Crawl"
- board text added: "REV: 1a"
- board text added: "Sensor Carousel"
