File: laser_carousel/carousel.sch (EAGLE design)
At the start: 52 parts

Commit message: More Board Committs
Parts:
- added FUD1, FUD2, FUD3, FUD4: FIDUCIAL, ENGI301:FIDUCIAL
- added MGT1, MGT2: MOUNTING_HOLE, ENGI301:MOUNTING_HOLE
- C12: device adafruit:C-US050-024X044 -> adafruit:C-US025-024X044
Connections:
- removed net N$10: C4.1, U$4.GND
- removed net N$4: C2.1, U$2.GND
- removed net N$7: C3.1, U$3.GND
- net GND: now also C2.1, C3.1, C4.1, U$2.GND, U$3.GND, U$4.GND
Changed lines of the file:
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@@
 <part name="U$12" library="ENGI301" deviceset="LASER_REC" device=""/>
 <part name="R12" library="adafruit" library_urn="urn:adsk.eagle:library:420" deviceset="R-US_" device="0204/2V" package3d_urn="urn:adsk.eagle:package:6240630/1" value="1k"/>
-<part name="C12" library="adafruit" library_urn="urn:adsk.eagle:library:420" deviceset="C-US" device="050-024X044" package3d_urn="urn:adsk.eagle:package:6240356/1" value="0.1uF"/>
+<part name="C12" library="adafruit" library_urn="urn:adsk.eagle:library:420" deviceset="C-US" device="025-024X044" package3d_urn="urn:adsk.eagle:package:6240324/1" value="0.1uF"/>
 <part name="U$13" library="ENGI301" deviceset="LASER_REC" device=""/>
 <part name="R13" library="adafruit" library_urn="urn:adsk.eagle:library:420" deviceset="R-US_" device="0204/2V" package3d_urn="urn:adsk.eagle:package:6240630/1" value="1k"/>
@@
 <part name="U$35" library="ENGI301" deviceset="VIN_5V" device=""/>
 <part name="JP2" library="adafruit" library_urn="urn:adsk.eagle:library:420" deviceset="PINHD-1X3" device="" package3d_urn="urn:adsk.eagle:package:6240710/1"/>
+<part name="GND17" library="ENGI301" deviceset="GND" device=""/>
+<part name="GND18" library="ENGI301" deviceset="GND" device=""/>
+<part name="GND19" library="ENGI301" deviceset="GND" device=""/>
+<part name="MGT1" library="ENGI301" deviceset="MOUNTING_HOLE" device=""/>
+<part name="MGT2" library="ENGI301" deviceset="MOUNTING_HOLE" device=""/>
+<part name="FUD1" library="ENGI301" deviceset="FIDUCIAL" device=""/>
+<part name="FUD2" library="ENGI301" deviceset="FIDUCIAL" device=""/>
+<part name="FUD3" library="ENGI301" deviceset="FIDUCIAL" device=""/>
+<part name="FUD4" library="ENGI301" deviceset="FIDUCIAL" device=""/>
 </parts>
 <sheets>
@@
 <attribute name="VALUE" x="62.23" y="104.14" size="1.778" layer="96"/>
 </instance>
+<instance part="GND17" gate="1" x="220.98" y="236.22" smashed="yes" rot="R90">
+<attribute name="VALUE" x="223.52" y="233.68" size="1.778" layer="96" rot="R90"/>
+</instance>
+<instance part="GND18" gate="1" x="276.86" y="236.22" smashed="yes" rot="R90">
+<attribute name="VALUE" x="279.4" y="233.68" size="1.778" layer="96" rot="R90"/>
+</instance>
+<instance part="GND19" gate="1" x="332.74" y="236.22" smashed="yes" rot="R90">
+<attribute name="VALUE" x="335.28" y="233.68" size="1.778" layer="96" rot="R90"/>
+</instance>
+<instance part="MGT1" gate="G$1" x="238.76" y="111.76" smashed="yes">
+<attribute name="NAME" x="239.522" y="109.728" size="1.27" layer="95"/>
+</instance>
+<instance part="MGT2" gate="G$1" x="254" y="111.76" smashed="yes">
+<attribute name="NAME" x="254.762" y="109.728" size="1.27" layer="95"/>
+</instance>
+<instance part="FUD1" gate="G$1" x="302.26" y="114.3" smashed="yes"/>
+<instance part="FUD2" gate="G$1" x="302.26" y="93.98" smashed="yes"/>
+<instance part="FUD3" gate="G$1" x="320.04" y="93.98" smashed="yes"/>
+<instance part="FUD4" gate="G$1" x="320.04" y="114.3" smashed="yes"/>
 </instances>
 <busses>
 </busses>
 <nets>
-<net name="N$4" class="0">
-<segment>
-<pinref part="U$2" gate="G$1" pin="GND"/>
-<pinref part="C2" gate="G$1" pin="1"/>
-<wire x1="195.58" y1="236.22" x2="203.2" y2="236.22" width="0.1524" layer="91"/>
-<junction x="203.2" y="236.22"/>
-<wire x1="203.2" y1="236.22" x2="218.44" y2="236.22" width="0.1524" layer="91"/>
-</segment>
-</net>
-<net name="N$7" class="0">
-<segment>
-<pinref part="U$3" gate="G$1" pin="GND"/>
-<pinref part="C3" gate="G$1" pin="1"/>
-<wire x1="251.46" y1="236.22" x2="259.08" y2="236.22" width="0.1524" layer="91"/>
-<junction x="259.08" y="236.22"/>
-<wire x1="259.08" y1="236.22" x2="274.32" y2="236.22" width="0.1524" layer="91"/>
-</segment>
-</net>
-<net name="N$10" class="0">
-<segment>
-<pinref part="U$4" gate="G$1" pin="GND"/>
-<pinref part="C4" gate="G$1" pin="1"/>
-<wire x1="307.34" y1="236.22" x2="314.96" y2="236.22" width="0.1524" layer="91"/>
-<junction x="314.96" y="236.22"/>
-<wire x1="314.96" y1="236.22" x2="330.2" y2="236.22" width="0.1524" layer="91"/>
-</segment>
-</net>
 <net name="VIN_5V" class="0">
 <segment>
@@
 <junction x="53.34" y="137.16"/>
 </segment>
+<segment>
+<pinref part="U$2" gate="G$1" pin="GND"/>
+<pinref part="C2" gate="G$1" pin="1"/>
+<wire x1="195.58" y1="236.22" x2="203.2" y2="236.22" width="0.1524" layer="91"/>
+<junction x="203.2" y="236.22"/>
+<wire x1="203.2" y1="236.22" x2="218.44" y2="236.22" width="0.1524" layer="91"/>
+<pinref part="GND17" gate="1" pin="GND"/>
+</segment>
+<segment>
+<pinref part="U$3" gate="G$1" pin="GND"/>
+<pinref part="C3" gate="G$1" pin="1"/>
+<wire x1="251.46" y1="236.22" x2="259.08" y2="236.22" width="0.1524" layer="91"/>
+<junction x="259.08" y="236.22"/>
+<wire x1="259.08" y1="236.22" x2="274.32" y2="236.22" width="0.1524" layer="91"/>
+<pinref part="GND18" gate="1" pin="GND"/>
+</segment>
+<segment>
+<pinref part="U$4" gate="G$1" pin="GND"/>
+<pinref part="C4" gate="G$1" pin="1"/>
+<wire x1="307.34" y1="236.22" x2="314.96" y2="236.22" width="0.1524" layer="91"/>
+<junction x="314.96" y="236.22"/>
+<wire x1="314.96" y1="236.22" x2="330.2" y2="236.22" width="0.1524" layer="91"/>
+<pinref part="GND19" gate="1" pin="GND"/>
+<junction x="330.2" y="236.22"/>
+</segment>
 </net>
